File: Candle_hw/Candle.kicad_pcb (KiCad board)
At the start: 2 copper layers, 13.8 x 74.4 mm, 58 parts, among them Q1 LED_RGB 5050, SW1 BUTTON, SW2 BUTTON, SW3 BUTTON

Commit message: + Candle05 hw
Parts:
- removed C22: 0.1u, Capacitors:CAP_0603
- removed C23, C24: *, Capacitors:CAP_0402
- removed L4: *, Inductors:IND_0402
- removed Q1: LED_RGB 5050, LEDs:LED_5050
- removed R6, R7: 4k7, Resistors:RES_0603
- removed XL7: CONN_4, Connectors:PLS-4
- added RP1: REFPOINT, PCB:REF_POINT_1MM, B.Cu at (126.5, 53.6)
- added RP2: REFPOINT, PCB:REF_POINT_1MM, F.Cu at (122.8, 75.8)
- added RP3: REFPOINT, PCB:REF_POINT_1MM, B.Cu at (134.7, 113.8)
- added RP4: REFPOINT, PCB:REF_POINT_1MM, F.Cu at (134.7, 113.8)
- ANT1: footprint Radio:ANT_868_10d4x36 -> Antennas:ANT_868_10d4x36
- C10: value 3.3pF -> 0.1u
- C12, C8: value 10n -> 0.1u
- C16, C6: value 220pF -> 0.1u
- C20: value 10u -> 0.1u
- DD2: value MMA8452Q -> LSM6DS3; footprint QFN_DFN:QFN16_5x3 -> LGA:14_3x2d5_p0d5
- R2: value 20k -> 56k
- R3, R4, R5: value 51R -> 100R
- XL1: footprint Connectors:PLS-6 -> Connectors:PLS-6-NoHole
- XL6: footprint Connectors:PLS-4 -> Connectors:PLS-4-Long
- moved C21 7.58 mm to (133.0, 93.1), turned to 0 degrees
- moved C20 7.01 mm to (133.0, 94.8), turned to 0 degrees
- moved XL6 3.89 mm to (128.7, 48.8)
- moved Logo1 2.60 mm to (128.5, 65.7)
- moved DD2 1.84 mm to (128.6, 94.0)
- moved TP2 1.15 mm to (125.7, 86.5)
- moved R4 0.40 mm to (123.6, 91.6)
- moved XL1 0.20 mm to (123.3, 107.3)
- moved R5 0.20 mm to (124.4, 88.4)
- turned SW3 to 180 degrees
Connections:
- ANT1 pad 1: /ANT2 -> /ANT1
- C20 pad 1: PwrMCU -> /ACC_PWR
- C21 pad 1: PwrMCU -> /ACC_PWR
- DD1 pad 11: (no net) -> /CC_GDO0
- DD1 pad 12: /CC_GDO2 -> /UART_TX
- DD1 pad 13: /CC_GDO0 -> /UART_RX
- DD1 pad 2: (no net) -> /ACC_INT1
- DD1 pad 25: (no net) -> /ACC_CS
- DD1 pad 26: (no net) -> /ACC_SCK
- DD1 pad 27: (no net) -> /ACC_MISO
- DD1 pad 28: (no net) -> /ACC_MOSI
- DD1 pad 30: /UART_TX -> /ACC_PWR
- DD1 pad 31: /UART_RX -> (no net)
- DD1 pad 38: (no net) -> /CC_GDO2
- DD1 pad 40: /ACC_INT1 -> (no net)
- DD1 pad 42: /I2C_SCL -> (no net)
- DD1 pad 43: /I2C_SDA -> (no net)
- DD2 pad 1: PwrMCU -> /ACC_MISO
- DD2 pad 10: GND -> (no net)
- DD2 pad 11: /ACC_INT1 -> (no net)
- DD2 pad 12: GND -> /ACC_CS
- DD2 pad 13: (no net) -> /ACC_SCK
- DD2 pad 14: PwrMCU -> /ACC_MOSI
- DD2 pad 2: Net-(C22-Pad1) -> GND
- DD2 pad 3: (no net) -> GND
- DD2 pad 4: /I2C_SCL -> /ACC_INT1
- DD2 pad 5: GND -> /ACC_PWR
- DD2 pad 6: /I2C_SDA -> GND
- DD2 pad 8: (no net) -> /ACC_PWR
Routing:
- net /ANT1: track 2.30 -> 86.3 mm
- net /ANT2: track 83.2 -> 0.00 mm
- net PwrMCU: track 90.9 -> 71.4 mm, vias 9 -> 6
- net /ACC_PWR: track 0.00 -> 15.5 mm, vias 0 -> 1
- net /UART_TX: track 2.18 -> 16.5 mm, vias 0 -> 2
- net /I2C_SCL: track 12.5 -> 0.00 mm, vias 2 -> 0
- net /I2C_SDA: track 11.8 -> 0.00 mm, vias 2 -> 0
- net GND: track 212.9 -> 203.4 mm, vias 35 -> 33
- net /ACC_INT1: track 6.83 -> 14.4 mm
- net Net-(Q1-Pad1): track 6.54 -> 0.00 mm
- net /ACC_CS: track 0.00 -> 5.68 mm, vias 0 -> 1
- net /UART_RX: track 6.64 -> 11.9 mm, vias 0 -> 2
- net Net-(DD1-Pad10): track 13.3 -> 18.1 mm
- net /ACC_SCK: track 0.00 -> 4.66 mm, vias 0 -> 1
- net Net-(C22-Pad1): track 4.38 -> 0.00 mm
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Other:
- board size 13.8 x 74.4 mm -> 13.8 x 68.9 mm
- board text added: "+"
- board text added: "Ostranna Candle 05"
- board text removed: "Candle 04"
